Commit message: first commit

File: sjtu_drone_description/urdf/sjtu_drone.urdf.xacro (robot description, xacro)
@@ -4,5 +4,5 @@
   <!-- Need argument to get from launch file -->
   <xacro:arg name="params_path" default="$(find sjtu_drone_bringup)/config/drone.yaml"/>
-  <!-- Need seperate property for xacro inorder processing -->
+  <!-- Need separate property for xacro inorder processing -->
   <xacro:property name="params_path" value="$(arg params_path)"/>
   <!-- Read in the yaml dict as mp (short for model parameters) -->
@@ -54,4 +54,10 @@
   </joint>
   <link name="bottom_cam_link"/>
+  <joint name="lidar_joint" type="fixed">
+    <origin rpy="0 0 0" xyz="0 0 0.1"/>
+    <parent link="base_link"/>
+    <child link="lidar_link"/>
+  </joint>
+  <link name="lidar_link"/>
   <gazebo>
     <plugin name='simple_drone' filename='libplugin_drone.so'>
@@ -284,3 +290,37 @@
     </sensor>
   </gazebo>
+  <!-- LiDAR sensor -->
+<gazebo reference="lidar_link">
+  <sensor name="lidar_sensor" type="ray">
+    <visualize>true</visualize>
+    <update_rate>10.0</update_rate>
+    <ray>
+      <scan>
+        <horizontal>
+          <samples>360</samples>
+          <resolution>1</resolution>
+          <min_angle>-3.14159</min_angle>
+          <max_angle>3.14159</max_angle>
+        </horizontal>
+      </scan>
+      <range>
+        <min>0.1</min>
+        <max>30.0</max>
+        <resolution>0.01</resolution>
+      </range>
+      <noise>
+        <type>gaussian</type>
+        <mean>0.0</mean>
+        <stddev>0.01</stddev>
+      </noise>
+    </ray>
+    <plugin name="gazebo_ros_ray_sensor" filename="libgazebo_ros_ray_sensor.so">
+      <ros>
+        <namespace>${mp['namespace']}</namespace>
+        <remapping>~/scan:=scan</remapping>
+      </ros>
+      <frame_name>${mp['namespace']}/lidar_link</frame_name>
+    </plugin>
+  </sensor>
+</gazebo>
 </robot>
